Commit message: add new box in xacro

File: urdf/mybot.xacro (robot description, xacro)
@@ -19,5 +19,5 @@
 	<xacro:property name="chassis_depth" value="0.2"/>
 	<xacro:property name="wheel_mass" value="5"/>
-	<xacro:property name="wheel_radius" value="0.2"/>
+	<xacro:property name="d" value="0.2"/>
 	<xacro:property name="wheel_length" value="0.05"/>
 	<xacro:property name="wheel_position" value="0.1"/>
@@ -26,4 +26,7 @@
 	<xacro:property name="camera_size" value="0.05"/>
 	<xacro:property name="camera_mass" value="0.1"/>
+	<xacro:property name="upperbox_height" value="0.375"/>
+	<xacro:property name="upperbox_width" value="0.5"/>
+	<xacro:property name="upperbox_depth" value="0.1"/>
 	<macro name="box_inertia" params="m x y z">
 	  	<inertia ixx="${m*(y*y+z*z)/12}" ixy = "0" ixz = "0"
@@ -43,5 +46,5 @@
 		   		<origin xyz="0 0 0" rpy="0 ${PI/2} ${PI/2}" />
 			    <geometry>
-			      	<cylinder length="${wheel_length}" radius="${wheel_radius}"/>
+			      	<cylinder length="${wheel_length}" radius="${d}"/>
 			    </geometry>
 		  	</collision>
@@ -49,5 +52,5 @@
 		    	<origin xyz="0 0 0" rpy="0 ${PI/2} ${PI/2}" />
 		    	<geometry>
-		      		<cylinder length="${wheel_length}" radius="${wheel_radius}"/>
+		      		<cylinder length="${wheel_length}" radius="${d}"/>
 		    	</geometry>
 		    	<material name="blue"/>
@@ -56,5 +59,5 @@
 		    	<origin xyz="0 0 0" rpy="0 ${PI/2} ${PI/2}" />
 		    	<mass value="${wheel_mass}"/>
-		    	<cylinder_inertia m="${wheel_mass}" r="${wheel_radius}" h="${wheel_length}"/>
+		    	<cylinder_inertia m="${wheel_mass}" r="${d}" h="${wheel_length}"/>
 		  	</inertial>
 		</link>
@@ -71,5 +74,5 @@
 			<origin xyz="${-0.2+chassis_height/2}
 						${tY * wheel_length/2 + tY*chassis_width/2}
-						${wheel_radius}" rpy="0 0 0" />
+						${d}" rpy="0 0 0" />
 		  	<axis xyz="0 1 0" rpy="0 0 0" />
 		  	<limit effort="100" velocity="100"/>
@@ -87,4 +90,19 @@
 		</transmission>
 	</macro>
+	<!-- <macro name="upper_body" params="">
+	</macro> -->
+	<link name="upper_body">
+		<visual>
+			<origin xyz="${chassis_height/4} 0 ${chassis_depth/2+d}" rpy="0 0 0"/>
+			<geometry>
+				<box size="${upperbox_height} ${upperbox_width} ${upperbox_depth}"/>
+			</geometry>
+			<material name="green"/>
+		</visual>
+	</link>
+	<joint name="upper_lower" type="fixed">
+		<parent link="chassis"/>
+		<child link="upper_body"/>
+	</joint>
 	<link name="base_link" />
 	<gazebo reference="chassis">
@@ -97,5 +115,5 @@
 	<link name="chassis">
 	  	<collision>
-	    	<origin xyz="0 0 ${wheel_radius}" rpy="0 0 0"/>
+	    	<origin xyz="0 0 ${d}" rpy="0 0 0"/>
 	    	<geometry>
 	      		<box size="${chassis_height} ${chassis_width} ${chassis_depth}"/>
@@ -103,5 +121,5 @@
 	  	</collision>
 	  	<visual>
-	    	<origin xyz="0 0 ${wheel_radius}" rpy="0 0 0"/>
+	    	<origin xyz="0 0 ${d}" rpy="0 0 0"/>
 	    	<geometry>
 	      		<box size="${chassis_height} ${chassis_width} ${chassis_depth}"/>
@@ -110,5 +128,5 @@
 	  	</visual>
 	  	<inertial>
-	    	<origin xyz="0 0 ${wheel_radius}" rpy="0 0 0"/>
+	    	<origin xyz="0 0 ${d}" rpy="0 0 0"/>
 	    	<mass value="${chassis_mass}"/>
 	    	<box_inertia m="${chassis_mass}" x="${chassis_height}" y="${chassis_width}"
@@ -123,5 +141,5 @@
 	  	<collision>
 	    <origin xyz="${casterRadius - chassis_height/2} 0
-	    			${casterRadius - chassis_depth + wheel_radius}" rpy="0 0 0"/>
+	    			${casterRadius - chassis_depth + d}" rpy="0 0 0"/>
 	    <geometry>
 	      	<sphere radius="${casterRadius}"/>
@@ -130,5 +148,5 @@
 	  <visual>
 	    	<origin xyz="${casterRadius - chassis_height/2} 0
-	    				${casterRadius - chassis_depth + wheel_radius}" rpy="0 0 0"/>
+	    				${casterRadius - chassis_depth + d}" rpy="0 0 0"/>
 	    <geometry>
 	      	<sphere radius="${casterRadius}"/>
@@ -138,5 +156,5 @@
 	  <inertial>
 	    <origin xyz="${casterRadius - chassis_height/2} 0
-	    			${casterRadius-chassis_depth + wheel_radius}" rpy="0 0 0"/>
+	    			${casterRadius-chassis_depth + d}" rpy="0 0 0"/>
 	    <mass value="${casterMass}"/>
 	    <sphere_inertia m="${casterMass}" r="${casterRadius}"/>
@@ -152,5 +170,5 @@
 	<joint name="camera_joint" type="fixed">
 	    <origin
-	    	xyz="${-2 * camera_size + chassis_height/2} 0 ${wheel_radius + chassis_depth / 2}"
+	    	xyz="${-2 * camera_size + chassis_height/2} 0 ${d + chassis_depth / 2}"
 	    	rpy="0 0 0"/>
 	    <parent link="chassis"/>
@@ -228,5 +246,5 @@
 		    <rightJoint>right_wheel_hinge</rightJoint>
 		    <wheelSeparation>${chassis_width+wheel_length}</wheelSeparation>
-		    <wheelDiameter>${2*wheel_radius}</wheelDiameter>
+		    <wheelDiameter>${2*d}</wheelDiameter>
 		    <broadcastTF>1</broadcastTF>
 			<wheelTorque>30</wheelTorque>

Commit message: finish complete robot xacro

File: urdf/mybot.xacro (robot description, xacro)
@@ -14,19 +14,19 @@
 	</material>
 	<xacro:property name="PI" value="3.1415926535897931"/>
-	<xacro:property name="chassis_mass" value="50"/>
-	<xacro:property name="chassis_width" value="0.5"/>
-	<xacro:property name="chassis_height" value="0.75"/>
-	<xacro:property name="chassis_depth" value="0.2"/>
+	<xacro:property name="chassis_mass" value="10"/>
+	<xacro:property name="chassis_width" value="0.2"/>
+	<xacro:property name="chassis_height" value="0.3"/>
+	<xacro:property name="chassis_depth" value="0.3"/>
 	<xacro:property name="wheel_mass" value="5"/>
 	<xacro:property name="d" value="0.2"/>
 	<xacro:property name="wheel_length" value="0.05"/>
 	<xacro:property name="wheel_position" value="0.1"/>
-	<xacro:property name="casterRadius" value="0.1"/>
+	<xacro:property name="casterRadius" value="${d-chassis_depth/2}"/>
 	<xacro:property name="casterMass" value="5"/>
 	<xacro:property name="camera_size" value="0.05"/>
 	<xacro:property name="camera_mass" value="0.1"/>
-	<xacro:property name="upperbox_height" value="0.375"/>
-	<xacro:property name="upperbox_width" value="0.5"/>
-	<xacro:property name="upperbox_depth" value="0.1"/>
+	<xacro:property name="upperbox_height" value="0.1"/>
+	<xacro:property name="upperbox_width" value="0.1"/>
+	<xacro:property name="upperbox_depth" value="0.3"/>
 	<macro name="box_inertia" params="m x y z">
 	  	<inertia ixx="${m*(y*y+z*z)/12}" ixy = "0" ixz = "0"
@@ -72,5 +72,5 @@
 		  	<parent link="chassis"/>
 		  	<child link="${lr}_wheel"/>
-			<origin xyz="${-0.2+chassis_height/2}
+			<origin xyz="${-chassis_height/4}
 						${tY * wheel_length/2 + tY*chassis_width/2}
 						${d}" rpy="0 0 0" />
@@ -90,9 +90,9 @@
 		</transmission>
 	</macro>
-	<!-- <macro name="upper_body" params="">
+	<!-- <macro name="upperbox" params="">
 	</macro> -->
-	<link name="upper_body">
+	<link name="upperbox">
 		<visual>
-			<origin xyz="${chassis_height/4} 0 ${chassis_depth/2+d}" rpy="0 0 0"/>
+			<origin xyz="0 0 0" rpy="0 0 0"/>
 			<geometry>
 				<box size="${upperbox_height} ${upperbox_width} ${upperbox_depth}"/>
@@ -102,6 +102,7 @@
 	</link>
 	<joint name="upper_lower" type="fixed">
+		<origin xyz="${chassis_height/4} 0 ${d+chassis_height/2+upperbox_depth/2}" rpy="0 0 0"/>
 		<parent link="chassis"/>
-		<child link="upper_body"/>
+		<child link="upperbox"/>
 	</joint>
 	<link name="base_link" />
@@ -139,7 +140,7 @@
 	</joint>
 	<link name="caster_wheel">
-	  	<collision>
-	    <origin xyz="${casterRadius - chassis_height/2} 0
-	    			${casterRadius - chassis_depth + d}" rpy="0 0 0"/>
+	  <collision>
+	    <origin xyz="${chassis_height/4} 0
+	    				${d-chassis_depth/2}" rpy="0 0 0"/>
 	    <geometry>
 	      	<sphere radius="${casterRadius}"/>
@@ -147,6 +148,6 @@
 	  </collision>
 	  <visual>
-	    	<origin xyz="${casterRadius - chassis_height/2} 0
-	    				${casterRadius - chassis_depth + d}" rpy="0 0 0"/>
+	    	<origin xyz="${chassis_height/4} 0
+	    				${d-chassis_depth/2}" rpy="0 0 0"/>
 	    <geometry>
 	      	<sphere radius="${casterRadius}"/>
@@ -155,6 +156,6 @@
 	  </visual>
 	  <inertial>
-	    <origin xyz="${casterRadius - chassis_height/2} 0
-	    			${casterRadius-chassis_depth + d}" rpy="0 0 0"/>
+	    <origin xyz="${chassis_height/4} 0
+	    				${d-chassis_depth/2}" rpy="0 0 0"/>
 	    <mass value="${casterMass}"/>
 	    <sphere_inertia m="${casterMass}" r="${casterRadius}"/>
@@ -170,12 +171,12 @@
 	<joint name="camera_joint" type="fixed">
 	    <origin
-	    	xyz="${-2 * camera_size + chassis_height/2} 0 ${d + chassis_depth / 2}"
+	    	xyz="0 0 0"
 	    	rpy="0 0 0"/>
-	    <parent link="chassis"/>
+	    <parent link="upperbox"/>
 	    <child link="camera"/>
 	</joint>
 	<link name="camera">
 	  	<collision>
-		    <origin xyz="0 0 0" rpy="0 0 0"/>
+		    <origin xyz="0 0 ${upperbox_depth/2}" rpy="0 0 0"/>
 		    <geometry>
 		      	<sphere radius="${camera_size}"/>
@@ -183,5 +184,5 @@
 	  	</collision>
 	  	<visual>
-		    <origin xyz="0 0 0" rpy="0 0 0"/>
+		    <origin xyz="0 0 ${upperbox_depth/2}" rpy="0 0 0"/>
 		    <geometry>
 		      	<sphere radius="${camera_size}"/>
@@ -191,5 +192,5 @@
 	  	<inertial>
 		    <mass value="${camera_mass}" />
-		    <origin xyz="0 0 0" rpy="0 0 0"/>
+		    <origin xyz="0 0 ${upperbox_depth/2}" rpy="0 0 0"/>
 		    <box_inertia m="${camera_mass}" x="${camera_size}" y="${camera_size}" z="${camera_size}"/>
 	  	</inertial>
